File: EAGLE_files/electrobassrev9_fix.sch (EAGLE design)
At the start: 290 parts, among them IC1 LMV324M, IC18 CY8C4124, IC2 4052D, IC3 LMV321M5, IC5 LMV321M5, J1 105162-0001, J2 SM06B-SRSS-TB(LF)(SN), J28 PJ-066A, J3 SM06B-SRSS-TB(LF)(SN), J5 SM06B-SRSS-TB(LF)(SN), J6 SM06B-SRSS-TB(LF)(SN), J7 SM06B-SRSS-TB(LF)(SN), J8 SM06B-SRSS-TB(LF)(SN), Q1 DMP3099L, U1 ES_DAISY_SEED_DOUBLE, U10 OPA1654, U2 LP2985, U3 MCP1755T-5002E/DCSOT-223_5_MC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, U4 CY8C5888LTI-LP097QFN-68-M, U5 ADUM3160BRWZRW_16_ADI-M, U6 LSM6DSLTR, U7 ES_DAISY_SEED_DOUBLE, U8 MCP23008T-E/SS, X1 3P-2MM-TH-MALE, X10 3P-2MM-TH-MALE, X11 3P-2MM-TH-MALE, X12 3P-2MM-TH-MALE, X13 3P-2MM-TH-MALE, X14 3P-2MM-TH-MALE, X15 3P-2MM-TH-MALE, X16 332-02, X17 332-02, X18 332-02, X19 332-02, X2 NRJ6HF2, X3 NRJ6HF2, X4 USB+SHIELD, X5 332-02, X6 332-02, X7 332-02, X8 332-02, X9 3P-2MM-TH-MALE

Commit message: fixed reading of new presets from plugin to align with electrosteel
Parts:
- added X20, X21: 3P-2MM-TH-MALE, CYCFI_Con:3P-2MM-TH-MALE
- added X22, X23: 332-02, con-garry:332-02
Connections:
- new net ELECTROSTEELHIGH: X20.3, X21.3
- new net ELECTROSTEEL_GND: X20.1, X20.2, X21.1, X21.2, X22-2.S, X23-2.S
- net AGND: now also JP1.6
- net AGND3: now also JP15.6
- net AGND4: no longer JP15.6
- net GNDINT: no longer JP1.6
Changed lines of the file:
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@@
 <attribute name="PARTNO" value="CC0603KRX7R8BB104"/>
 </part>
+<part name="V1" library="custom" deviceset="AGND3" device=""/>
+<part name="X20" library="CYCFI_Con" deviceset="3P-2MM-TH-MALE" device="">
+<attribute name="PARTNO" value="*DNP"/>
+</part>
+<part name="X21" library="CYCFI_Con" deviceset="3P-2MM-TH-MALE" device="">
+<attribute name="PARTNO" value="*DNP"/>
+</part>
+<part name="X22" library="con-garry" library_urn="urn:adsk.eagle:library:147" deviceset="332-02" device="" package3d_urn="urn:adsk.eagle:package:6810/1">
+<attribute name="PARTNO" value="*DNP"/>
+</part>
+<part name="X23" library="con-garry" library_urn="urn:adsk.eagle:library:147" deviceset="332-02" device="" package3d_urn="urn:adsk.eagle:package:6810/1">
+<attribute name="PARTNO" value="*DNP"/>
+</part>
 </parts>
 <sheets>
@@
 <pinref part="JP1" gate="A" pin="7"/>
 <wire x1="421.64" y1="-76.2" x2="431.8" y2="-76.2" width="0.1524" layer="91"/>
+<wire x1="431.8" y1="-76.2" x2="436.118" y2="-76.2" width="0.1524" layer="91"/>
+<wire x1="436.118" y1="-76.2" x2="436.118" y2="-73.66" width="0.1524" layer="91"/>
+<junction x="431.8" y="-76.2"/>
+<pinref part="JP1" gate="A" pin="6"/>
+<wire x1="436.118" y1="-73.66" x2="439.42" y2="-73.66" width="0.1524" layer="91"/>
 </segment>
 </net>
@@
 <pinref part="GND7" gate="G$1" pin="GNDINT"/>
 <wire x1="439.42" y1="-71.12" x2="464.82" y2="-71.12" width="0.1524" layer="91"/>
-<pinref part="JP1" gate="A" pin="6"/>
-<wire x1="439.42" y1="-73.66" x2="439.42" y2="-71.12" width="0.1524" layer="91"/>
-<junction x="439.42" y="-71.12"/>
 </segment>
 <segment>
@@
 <attribute name="VALUE" x="446.405" y="-83.82" size="1.778" layer="96" ratio="12"/>
 </instance>
+<instance part="V1" gate="G$1" x="482.6" y="-76.2" smashed="yes">
+<attribute name="VALUE" x="479.425" y="-78.74" size="1.778" layer="96" ratio="12"/>
+</instance>
 </instances>
 <busses>
@@
 <wire x1="449.58" y1="-76.2" x2="449.58" y2="-78.74" width="0.1524" layer="91"/>
 </segment>
+<segment>
+<pinref part="JP15" gate="A" pin="6"/>
+<pinref part="V1" gate="G$1" pin="AGND3"/>
+<wire x1="472.44" y1="-73.66" x2="482.6" y2="-73.66" width="0.1524" layer="91"/>
+</segment>
 </net>
 <net name="DGND3" class="0">
@@
 <wire x1="472.44" y1="-71.12" x2="505.46" y2="-71.12" width="0.1524" layer="91"/>
 <wire x1="505.46" y1="-71.12" x2="505.46" y2="-50.8" width="0.1524" layer="91"/>
-<pinref part="JP15" gate="A" pin="6"/>
-<wire x1="472.44" y1="-73.66" x2="472.44" y2="-71.12" width="0.1524" layer="91"/>
-<junction x="472.44" y="-71.12"/>
 </segment>
 </net>
@@
 </segment>
 </net>
+</nets>
+</sheet>
+<sheet>
+<plain>
+</plain>
+<instances>
+<instance part="X20" gate="G$1" x="2.54" y="91.44" smashed="yes">
+<attribute name="PARTNO" x="2.54" y="91.44" size="1.778" layer="96" display="off"/>
+<attribute name="VALUE" x="1.27" y="83.82" size="1.778" layer="96"/>
+<attribute name="NAME" x="1.27" y="97.282" size="1.778" layer="95"/>
+</instance>
+<instance part="X21" gate="G$1" x="2.54" y="71.12" smashed="yes">
+<attribute name="PARTNO" x="2.54" y="71.12" size="1.778" layer="96" display="off"/>
+<attribute name="VALUE" x="1.27" y="63.5" size="1.778" layer="96"/>
+<attribute name="NAME" x="1.27" y="76.962" size="1.778" layer="95"/>
+</instance>
+<instance part="X22" gate="-1" x="40.64" y="91.44" smashed="yes">
+<attribute name="PARTNO" x="40.64" y="91.44" size="1.778" layer="96" display="off"/>
+<attribute name="NAME" x="43.18" y="90.678" size="1.524" layer="95"/>
+<attribute name="VALUE" x="39.878" y="92.837" size="1.778" layer="96"/>
+</instance>
+<instance part="X22" gate="-2" x="60.96" y="91.44" smashed="yes">
+<attribute name="NAME" x="63.5" y="90.678" size="1.524" layer="95"/>
+<attribute name="VALUE" x="60.198" y="92.837" size="1.778" layer="96"/>
+</instance>
+<instance part="X23" gate="-1" x="40.64" y="71.12" smashed="yes">
+<attribute name="PARTNO" x="40.64" y="71.12" size="1.778" layer="96" display="off"/>
+<attribute name="NAME" x="43.18" y="70.358" size="1.524" layer="95"/>
+</instance>
+<instance part="X23" gate="-2" x="60.96" y="71.12" smashed="yes">
+<attribute name="NAME" x="63.5" y="70.358" size="1.524" layer="95"/>
+<attribute name="VALUE" x="60.198" y="72.517" size="1.778" layer="96"/>
+</instance>
+</instances>
+<busses>
+</busses>
+<nets>
+<net name="ELECTROSTEEL_GND" class="0">
+<segment>
+<pinref part="X23" gate="-2" pin="S"/>
+<wire x1="58.42" y1="71.12" x2="58.42" y2="66.04" width="0.1524" layer="91"/>
+<pinref part="X21" gate="G$1" pin="1"/>
+<wire x1="58.42" y1="66.04" x2="10.16" y2="66.04" width="0.1524" layer="91"/>
+<wire x1="10.16" y1="66.04" x2="10.16" y2="68.58" width="0.1524" layer="91"/>
+<pinref part="X21" gate="G$1" pin="2"/>
+<wire x1="10.16" y1="68.58" x2="10.16" y2="71.12" width="0.1524" layer="91"/>
+<junction x="10.16" y="68.58"/>
+<label x="10.16" y="66.04" size="1.778" layer="95"/>
+</segment>
+<segment>
+<pinref part="X20" gate="G$1" pin="1"/>
+<pinref part="X22" gate="-2" pin="S"/>
+<wire x1="10.16" y1="88.9" x2="58.42" y2="88.9" width="0.1524" layer="91"/>
+<wire x1="58.42" y1="88.9" x2="58.42" y2="91.44" width="0.1524" layer="91"/>
+<pinref part="X20" gate="G$1" pin="2"/>
+<wire x1="10.16" y1="91.44" x2="10.16" y2="88.9" width="0.1524" layer="91"/>
+<junction x="10.16" y="88.9"/>
+<label x="12.7" y="88.9" size="1.778" layer="95"/>
+</segment>
+</net>
+<net name="ELECTROSTEELHIGH" class="0">
+<segment>
+<pinref part="X21" gate="G$1" pin="3"/>
+<wire x1="10.16" y1="73.66" x2="10.16" y2="78.74" width="0.1524" layer="91"/>
+<label x="10.16" y="78.74" size="1.778" layer="95"/>
+</segment>
+<segment>
+<pinref part="X20" gate="G$1" pin="3"/>
+<wire x1="10.16" y1="93.98" x2="10.16" y2="99.06" width="0.1524" layer="91"/>
+<label x="10.16" y="99.06" size="1.778" layer="95"/>
+</segment>
+</net>
