File: EAGLE_files/rev10/electrobassrev10_fix_2.kicad_pcb (KiCad board)
At the start: 4 copper layers, 346.6 x 245.1 mm, 295 parts, among them IC1 LMV324M, IC2 1253S08-U, IC3 LMV321M5, IC4 CY8C58LPXXX_USB_4JTAG, IC5 LMV321M5, IC6 1253S08-U, IC7 1253S08-U, IC8 1253S08-U, J1 105162-0001, J10 4P-2.0, J11 4P-2.0, J13 4P-2.0, J2 SM06B-SRSS-TB(LF)(SN), J28 PJ-066A, J3 SM06B-SRSS-TB(LF)(SN), J31 4P-2.0-90D, J4 4P-2.0, J5 SM06B-SRSS-TB(LF)(SN), J6 SM06B-SRSS-TB(LF)(SN), J7 SM06B-SRSS-TB(LF)(SN), J8 SM06B-SRSS-TB(LF)(SN), J9 4P-2.0, Q1 DMP3099L, U1 ES_DAISY_SEED_DOUBLE, U10 DG403DVZTSSOP16_4P50X5P10_INR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, U11 MC74HC4052ADTR2GTSSOP-16_ONS-L, U12 DG403DVZTSSOP16_4P50X5P10_INR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, U13 ES_DAISY_SEED_DOUBLE, U14 CY8C4024AZI-S413TQFP_24AZI-S4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, U15 DG403DVZTSSOP16_4P50X5P10_INR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, U16 DG403DVZTSSOP16_4P50X5P10_INR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, U2 LP2985, U3 OPA1664AIPWRPW14_TEX-L, U4 ES_DAISY_SEED_DOUBLE, U5 ADUM3160BRWZRW_16_ADI-M, U6 LSM6DSLTR, U7 ES_DAISY_SEED_DOUBLE, U8 MCP23008T-E/SS, U9 MC74HC4052ADTR2GTSSOP-16_ONS-L, X1 3P-2MM-TH-MALE, X10 3P-2MM-TH-MALE, X11 3P-2MM-TH-MALE, X12 3P-2MM-TH-MALE, X13 3P-2MM-TH-MALE, X14 3P-2MM-TH-MALE, X15 3P-2MM-TH-MALE, X16 332-02, X17 332-02, X18 332-02, X19 332-02, X2 NRJ6HF2, X3 NRJ6HF2, X4 USB+SHIELD, X5 332-02, X6 332-02, X7 332-02, X8 332-02, X9 3P-2MM-TH-MALE

Commit message: added new electrobass revision kicad files
Parts:
- removed C15, C16, C17, C18, C19, C20, C21, C22, C23, C24, C25, C28: .1uf, electrobassrev10_fix_2:C0603K
- removed C35, C37, C67, C68: 10uf, electrobassrev10_fix_2:C1206K
- removed D14: , electrobassrev10_fix_2:LED-1206-BOTTOM_529
- removed IC2, IC6, IC7, IC8: 1253S08-U, electrobassrev10_fix_2:SOIC127P600X173-8N
- removed L2: 2.2uH, electrobassrev10_fix_2:BOURNS_SRP2010
- removed PS1: UWE1215S-3WR3, electrobassrev10_fix_2:CONV_UWE1215S-3WR3
- removed R64: 47R, electrobassrev10_fix_2:R0603_334
- removed U10, U12, U15, U16: DG403DVZTSSOP16_4P50X5P10_INR-L, electrobassrev10_fix_2:TSSOP16_4P50X5P10_INR-L
- removed U13, U4, U7, U_12: ES_DAISY_SEED_DOUBLE, electrobassrev10_fix_2:ES_DAISY_SEED_DOUBLE
- removed UNK12VD1: , electrobassrev10_fix_2:1X01
- removed UNK600R0: 10k, electrobassrev10_fix_2:R0603
- removed UNK_HOLE_0: , electrobassrev10_fix_2:dummyfp0
- removed UNK_HOLE_1: , electrobassrev10_fix_2:dummyfp1
- removed UNK_HOLE_10: , electrobassrev10_fix_2:dummyfp10
- removed UNK_HOLE_11: , electrobassrev10_fix_2:dummyfp11
- removed UNK_HOLE_12: , electrobassrev10_fix_2:dummyfp12
- removed UNK_HOLE_13: , electrobassrev10_fix_2:dummyfp13
- removed UNK_HOLE_14: , electrobassrev10_fix_2:dummyfp14
- removed UNK_HOLE_2: , electrobassrev10_fix_2:dummyfp2
- removed UNK_HOLE_3: , electrobassrev10_fix_2:dummyfp3
- removed UNK_HOLE_4: , electrobassrev10_fix_2:dummyfp4
- removed UNK_HOLE_5: , electrobassrev10_fix_2:dummyfp5
- removed UNK_HOLE_6: , electrobassrev10_fix_2:dummyfp6
- removed UNK_HOLE_7: , electrobassrev10_fix_2:dummyfp7
- removed UNK_HOLE_8: , electrobassrev10_fix_2:dummyfp8
- removed UNK_HOLE_9: , electrobassrev10_fix_2:dummyfp9
- added A10: Electrosmith_Daisy_Seed_Rev4, Module:Electrosmith_Daisy_Seed, F.Cu at (217.4, 97.5)
- added A2: Electrosmith_Daisy_Seed_Rev4, Module:Electrosmith_Daisy_Seed, F.Cu at (218.6, 51.1)
- added A3: Electrosmith_Daisy_Seed_Rev4, Module:Electrosmith_Daisy_Seed, F.Cu at (242.4, 25.1)
- added A6: Electrosmith_Daisy_Seed_Rev4, Module:Electrosmith_Daisy_Seed, F.Cu at (218.3, 74.9)
- added C100: .1uf, Capacitor_SMD:C_0603_1608Metric, F.Cu at (329.2, 59.8)
- added C102: .1uf, Capacitor_SMD:C_0402_1005Metric, F.Cu at (268.7, 78.7)
- added C103: EEE-HP1E220P, Snapeda:CAP_PAN_EEE_D_PAN-L, F.Cu at (287.8, 96.6)
- added C104: .1uf, Capacitor_SMD:C_0402_1005Metric, F.Cu at (279.9, 78.7)
- added C105: .1uf, Capacitor_SMD:C_0402_1005Metric, F.Cu at (276.6, 68.1)
- added C106: .1uf, Capacitor_SMD:C_0402_1005Metric, F.Cu at (283.2, 62.7)
- added C3: .1uf, Capacitor_SMD:C_0603_1608Metric, F.Cu at (333.5, 39.6)
- added C69: .1uf, Capacitor_SMD:C_0603_1608Metric, F.Cu at (333.8, 42.7)
- added C71: .1uf, Capacitor_SMD:C_0603_1608Metric, F.Cu at (333.8, 45.5)
- added C72: 100pf, Capacitor_SMD:C_0603_1608Metric, F.Cu at (333.8, 48.5)
- added C73: 33nf, Capacitor_SMD:C_1206_3216Metric, F.Cu at (293.1, 80.8)
- added C74: 47nf, Capacitor_SMD:C_0603_1608Metric, F.Cu at (325.2, 67.4)
- added C75: 100pf, Capacitor_SMD:C_0603_1608Metric, F.Cu at (325.2, 69.9)
- added C76: 100pf, Capacitor_SMD:C_0603_1608Metric, F.Cu at (333.8, 36.1)
- added C77: 1uf, Capacitor_SMD:CP_Elec_5x5.9, F.Cu at (328.2, 78.0)
- added C78: 22nf, Capacitor_SMD:C_1206_3216Metric, F.Cu at (315.4, 77.4)
- added C83: 10000pf Y2, Capacitor_THT:C_Rect_L13.0mm_W6.0mm_P10.00mm_FKS3_FKP3_MKS4, F.Cu at (286.4, 114.9)
- added C89: 2.2uf, Capacitor_SMD:CP_Elec_6.3x4.9, F.Cu at (315.7, 56.1)
- added C90: 2.2uf, Capacitor_SMD:CP_Elec_6.3x4.9, F.Cu at (315.5, 67.8)
- added C91: .1uf, Capacitor_SMD:C_0402_1005Metric, F.Cu at (293.6, 91.4)
- added C92: .1uf, Capacitor_SMD:C_0402_1005Metric, F.Cu at (268.0, 55.4)
- added C96: .1uf, Capacitor_SMD:C_0402_1005Metric, F.Cu at (303.8, 87.9)
- added C97: .1uf, Capacitor_SMD:C_0402_1005Metric, F.Cu at (279.7, 55.4)
- added D15: WL-SMRW_1206_REC, Snapeda:WL-SMRW_1206_REC, F.Cu at (224.9, -2.83)
- added J12: MEM2075-00-140-01-A, Snapeda:GCT_MEM2075-00-140-01-A, F.Cu at (204.2, 86.8)
- added J18: 110990030, Connector:NS-Tech_Grove_1x04_P2mm_Vertical, F.Cu at (293.7, 120.7)
- added R100: 470k, Resistor_SMD:R_0603_1608Metric, F.Cu at (333.2, 59.8)
- added R101: 33k, Resistor_SMD:R_0603_1608Metric, F.Cu at (333.2, 62.3)
- added R102: 47k, Resistor_SMD:R_0603_1608Metric, F.Cu at (333.2, 64.9)
- added R104: 10k, Resistor_SMD:R_0402_1005Metric, F.Cu at (273.1, 69.6)
- added R105: 10k, Resistor_SMD:R_0402_1005Metric, F.Cu at (273.1, 62.7)
- added R106: 47R, electrobassrev10_fix_2:R0603, F.Cu at (242.6, 102.9)
- added R112: 10k, Resistor_SMD:R_0402_1005Metric, F.Cu at (276.4, 64.8)
- added R113: 0R, Resistor_SMD:R_0603_1608Metric, F.Cu at (280.4, 29.0)
- added R114: 1k, Resistor_SMD:R_0603_1608Metric, F.Cu at (333.2, 67.4)
- added R115: 0R, Resistor_SMD:R_0603_1608Metric, F.Cu at (283.2, 29.0)
- added R116: 560R, Resistor_SMD:R_0402_1005Metric_Pad0.72x0.64mm_HandSolder, F.Cu at (292.1, 105.7)
- added R117: 100R, Resistor_SMD:R_0402_1005Metric, F.Cu at (279.7, 91.4)
- added R150: 1M, Resistor_SMD:R_1206_3216Metric, F.Cu at (280.8, 103.4)
- added R32: 0R, Resistor_SMD:R_0603_1608Metric, F.Cu at (253.0, 101.1)
- added R34: 1M, Resistor_SMD:R_0603_1608Metric, F.Cu at (329.2, 62.3)
- added R36: 470k, Resistor_SMD:R_0603_1608Metric, F.Cu at (329.2, 64.9)
- added R57: 1k, Resistor_SMD:R_0603_1608Metric, F.Cu at (329.2, 67.4)
- added R59: 10k, Resistor_SMD:R_0603_1608Metric, F.Cu at (329.2, 69.9)
- added R66: 47k, Resistor_SMD:R_0603_1608Metric, F.Cu at (333.2, 57.3)
- added R67: 0R, Resistor_SMD:R_0603_1608Metric, F.Cu at (255.5, 102.1)
- added R68: 0R, Resistor_SMD:R_0603_1608Metric, F.Cu at (258.3, 102.1)
- added R87: 2K, Resistor_SMD:R_0402_1005Metric_Pad0.72x0.64mm_HandSolder, F.Cu at (245.9, 102.6)
- added R88: 2K, Resistor_SMD:R_0402_1005Metric_Pad0.72x0.64mm_HandSolder, F.Cu at (248.2, 102.6)
- added R89: 0R, Resistor_SMD:R_0603_1608Metric, F.Cu at (253.2, 78.0)
- added R90: 0R, Resistor_SMD:R_0603_1608Metric, F.Cu at (259.1, 78.7)
- added R91: 0R, Resistor_SMD:R_0603_1608Metric, F.Cu at (256.8, 54.9)
- added R92: 0R, Resistor_SMD:R_0603_1608Metric, F.Cu at (259.8, 54.9)
- added R98: 10k, Resistor_SMD:R_0402_1005Metric, F.Cu at (273.1, 67.3)
- added R99: 10k, Resistor_SMD:R_0402_1005Metric, F.Cu at (273.1, 65.0)
- added RV1: 50k, Potentiometer_THT:Potentiometer_Bourns_3266Y_Vertical, F.Cu at (294.1, 110.1)
- added RV2: 50k, Potentiometer_THT:Potentiometer_Bourns_3266Y_Vertical, F.Cu at (280.8, 94.0)
- added S1: TL1105SPF160Q, Snapeda:SW_TL1105SPF160Q, F.Cu at (30.1, 135.0)
- added S3: TL1105SPF160Q, Snapeda:SW_TL1105SPF160Q, F.Cu at (16.9, 137.7)
- added S5: TL1105SPF160Q, Snapeda:SW_TL1105SPF160Q, F.Cu at (3.43, 137.3)
- added S6: TL1105SPF160Q, Snapeda:SW_TL1105SPF160Q, F.Cu at (-24.7, 132.1)
- added SW1: B3F-1025, UltraLibrarian:B3F-1025, F.Cu at (268.1, 103.7)
- added TP0: TestPoint, Connector_Pin:Pin_D0.9mm_L10.0mm_W2.4mm_FlatFork, F.Cu at (255.5, 93.7)
- added TP1: TestPoint, Connector_Pin:Pin_D0.9mm_L10.0mm_W2.4mm_FlatFork, F.Cu at (256.3, 71.4)
- added TP2: TestPoint, Connector_Pin:Pin_D0.9mm_L10.0mm_W2.4mm_FlatFork, F.Cu at (258.6, 45.7)
- added TP3: TestPoint, Connector_Pin:Pin_D0.9mm_L10.0mm_W2.4mm_FlatFork, F.Cu at (280.4, 20.8)
- added U17: NJM4580, Snapeda:NJR-SOP8_NJR-L, F.Cu at (300.5, 79.2)
- added U18: MCP45HV51T-503E/ST, Snapeda:TSSOP14_MC_MCH-L, F.Cu at (303.3, 38.4)
- added U19: MCP45HV51T-503E/ST, Snapeda:TSSOP14_MC_MCH-L, F.Cu at (296.8, 38.4)
- added U20: MCP45HV51T-503E/ST, Snapeda:TSSOP14_MC_MCH-L, F.Cu at (290.3, 38.4)
- added U21: MCP45HV51T-503E/ST, Snapeda:TSSOP14_MC_MCH-L, F.Cu at (283.8, 38.4)
- added U23: INA2134UA, footprints:D14-M, F.Cu at (273.8, 55.4)
- added U24: INA2134UA, footprints:D14-M, F.Cu at (274.3, 78.7)
- added U28: OPA1642AIDR, footprints:D8, F.Cu at (281.4, 66.5)
- added U29: DRV135UA/2K5, footprints:D0008A_N, F.Cu at (274.8, 95.8)
- A1, AGND5, CP1, CP2, CP3, CP4, DGND0, DGND1, G1, KNOB1, KNOB2, SC0, SD0, ST1, ST2, ST3, ST4, UNK10VA0, UNK12VD0, VT1, VT2, VT3, VT4: value (none) -> PINHD-1X1
- CV_PEDAL0, VBUS0: value (none) -> PINHD-1X1; footprint electrobassrev10_fix_2:1X01_325 -> electrobassrev10_fix_2:1X01
- D10, D11, D12, D4, D5, D6, D7, D8: value (none) -> WL-SMRW_1206_REC; footprint electrobassrev10_fix_2:LED-1206-BOTTOM_529 -> Snapeda:WL-SMRW_1206_REC
- D13: value (none) -> LED1206-BOTTOM
- D20: value MBRS340T3 -> MBRS30T3
- IC1: value LMV324M -> LMV324?M
- IC3, IC5: value LMV321M5 -> LMV321?M5
- J1: value 105162-0001 -> Conn_01x02_Pin; footprint electrobassrev10_fix_2:105162-0001 -> Connector_PinHeader_2.54mm:PinHeader_1x02_P2.54mm_Vertical
- JP1, JP15, JP2: value (none) -> PINHD-2X8
- JP37: value (none) -> PINHD-1X4
- L5: value (none) -> L-US6000-XXX-RC
- LED1: value (none) -> LEDCHIP-LED0603
- R137, R19, R192, R193, R194, R199, R4: footprint electrobassrev10_fix_2:R0603_16378527 -> electrobassrev10_fix_2:R0603
- R2, R3, R37, R38, R39, R40, R41, R45, R46, R5, R6, R60, R61, R62, R63, R7, R9: footprint electrobassrev10_fix_2:R0603_334 -> electrobassrev10_fix_2:R0603
- R23, R27, R28: footprint electrobassrev10_fix_2:R0603 -> Resistor_SMD:R_0402_1005Metric
- R29, R30: value 10k -> 0R; footprint electrobassrev10_fix_2:R0603 -> Resistor_SMD:R_0603_1608Metric
- R31: value 5R -> 0R; footprint electrobassrev10_fix_2:R0603 -> Resistor_SMD:R_0603_1608Metric
- R47, R51, R52, R53: value (none) -> R-TRIMM3314J
- U3: value OPA1664AIPWRPW14_TEX-L -> OPA1642AIDR; footprint electrobassrev10_fix_2:PW14_TEX-L -> footprints:D8
- moved R31 93.3 mm to (277.1, 28.2)
- moved R30 84.1 mm to (253.7, 54.9), turned to 0 degrees
- moved R29 67.1 mm to (256.3, 78.7), turned to 90 degrees
- moved J1 58.9 mm to (296.5, 114.6), turned to 90 degrees
- moved U3 42.0 mm to (299.0, 90.2)
- moved R96 39.2 mm to (219.7, 91.9), turned to 90 degrees
- moved R94 38.6 mm to (227.8, 92.2), turned to 90 degrees
- moved R97 38.6 mm to (222.2, 91.9), turned to 90 degrees
- moved R93 37.9 mm to (225.0, 91.9), turned to 90 degrees
- moved UNK12VD0 37.6 mm to (253.0, 123.7), turned to 0 degrees
- moved R95 35.3 mm to (230.4, 92.2), turned to 90 degrees
- moved R27 32.5 mm to (293.1, 93.5), turned to 0 degrees
- moved R5 30.6 mm to (232.7, 102.4)
- moved R7 30.6 mm to (225.0, 102.4)
- moved R2 30.5 mm to (220.1, 102.1)
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Connections:
- net +5V_ISOL renamed /electrobassrev10_fix_2_1/ADC1OPAMPOUT
- net 1.5V_MID renamed /electrobassrev10_fix_2_1/1.5V_MID
- net 12VD1 renamed +12V
- net 12VIN renamed /electrobassrev10_fix_2_1/12VIN
- net 3V3D5 renamed /electrobassrev10_fix_2_3/FR_3V3
- net 3V3FORPEDAL renamed Net-(JP1-Pad9)
- net ADC2OPAMPOUT renamed Net-(U5-UD-)
- net ADC3OPAMPOUT renamed /electrobassrev10_fix_2_6/AGND4
- net ADC4OPAMPOUT renamed /electrobassrev10_fix_2_1/ADC3OPAMPOUT
- net AGND4 renamed Net-(U5-DD-)
- net BLUE_LED renamed /electrobassrev10_fix_2_1/BLUE_LED
- net BYPASS renamed Net-(U2-BYPASS)
- net CAP_0_0 renamed /electrobassrev10_fix_2_1/CAP_0_0
- net CAP_0_1 renamed /electrobassrev10_fix_2_1/CAP_0_1
- net CAP_0_2 renamed /electrobassrev10_fix_2_1/CAP_0_2
- net CAP_0_3 renamed /electrobassrev10_fix_2_1/CAP_0_3
- net CAP_1_0 renamed /electrobassrev10_fix_2_1/CAP_1_0
- net CAP_1_1 renamed /electrobassrev10_fix_2_1/CAP_1_1
- net CAP_1_2 renamed /electrobassrev10_fix_2_1/CAP_1_2
- net CAP_1_3 renamed /electrobassrev10_fix_2_1/CAP_1_3
- net CMOD_CH0 renamed Net-(IC4-P1_6)
- net CMOD_CH1 renamed Net-(IC4-P0_2)
- net CV_PEDAL renamed /electrobassrev10_fix_2_1/CV_PEDAL
- net CV_PEDAL_SENSE renamed /electrobassrev10_fix_2_1/CV_PEDAL_SENSE
- net DM renamed /electrobassrev10_fix_2_1/DM
- net DOWN renamed /electrobassrev10_fix_2_1/DOWN
- net DP renamed /electrobassrev10_fix_2_1/DP
- net EGND renamed /electrobassrev10_fix_2_3/FR_GND
- net ENTER renamed Net-(U8-GP0)
- net EXT_MUX_EN renamed /electrobassrev10_fix_2_1/EXT_MUX_EN
- net EXT_MUX_EN2 renamed Net-(IC4-P12_5)
- net EXT_MUX_S0 renamed /electrobassrev10_fix_2_1/EXT_MUX_S0
- net EXT_MUX_S1 renamed /electrobassrev10_fix_2_1/EXT_MUX_S1
- net FR_3V3 renamed /electrobassrev10_fix_2_3/SCL_1
- net FR_GND renamed /electrobassrev10_fix_2_3/SDA_1
- net GNDINT_KNOBS renamed Net-(U5-UD+)
- net IDAC_OUT renamed /electrobassrev10_fix_2_1/IDAC_OUT
- net JOY_X renamed /electrobassrev10_fix_2_1/JOY_X
- net JOY_Y renamed /electrobassrev10_fix_2_1/JOY_Y
- net KNOB_1 renamed /electrobassrev10_fix_2_1/KNOB_1
- net KNOB_2 renamed /electrobassrev10_fix_2_1/KNOB_2
- net MISO_1 renamed /electrobassrev10_fix_2_1/MISO_1
- net MISO_1_P renamed Net-(R63-Pad1)
- net MOSI_1 renamed /electrobassrev10_fix_2_1/MOSI_1
- net MOSI_2_P renamed Net-(IC4-P12_4)
- net N$23 renamed /electrobassrev10_fix_2_1/USBDP
- net N$24 renamed /electrobassrev10_fix_2_1/USBDM
- net N$48 renamed /electrobassrev10_fix_2_5/O_SCL
- net N$60 renamed /electrobassrev10_fix_2_7/PICKUP1_OUT
- net N$61 renamed /electrobassrev10_fix_2_7/PICKUP4_OUT
- net N$62 renamed /electrobassrev10_fix_2_1/ENTER
- net N$63 renamed /electrobassrev10_fix_2_1/PROG_RESET
- net N$64 renamed /electrobassrev10_fix_2_1/PROG_SWDIO
- net N$65 renamed /electrobassrev10_fix_2_1/NECKSENSE1
- net N$66 renamed /electrobassrev10_fix_2_1/NECKSENSE2
- net N$75 renamed /electrobassrev10_fix_2_1/EXT_MUX_EN2
- net N$82 renamed /electrobassrev10_fix_2_1/NECKSENSE3
- net N$83 renamed /electrobassrev10_fix_2_1/NECKSENSE4
- net N$84 renamed /electrobassrev10_fix_2_1/CMOD_CH0
- net N$91 renamed /electrobassrev10_fix_2_1/AUDIO_L_PREKNOB
- net N$92 renamed /electrobassrev10_fix_2_1/AUDIO_L_POSTKNOB
- net N$93 renamed /electrobassrev10_fix_2_1/AUDIO_R_POSTKNOB
- net N$94 renamed /electrobassrev10_fix_2_1/AUDIO_R_PREKNOB
- net NECKSENSE1 renamed Net-(U8-GP1)
- net NECKSENSE2 renamed Net-(U8-GP4)
- net NECKSENSE3 renamed /electrobassrev10_fix_2_1/CMOD_CH1
- net NECKSENSE4 renamed Net-(IC4-P1_5)
- net O_CB1 renamed /electrobassrev10_fix_2_5/O_CB3
- net O_CB2 renamed Net-(JP10-P$1)
- net O_CB3 renamed Net-(A1-Pad1)
- net O_GND renamed Net-(JP15-Pad5)
- net O_SCL renamed /electrobassrev10_fix_2_5/O_CB1
- net O_SDA renamed /electrobassrev10_fix_2_5/O_CB2
- net PICKUP1 renamed /electrobassrev10_fix_2_1/PICKUP1
- net PICKUP1_OUT renamed /electrobassrev10_fix_2_7/PICKUP_PWR1
- net PICKUP1_OUT2 renamed /electrobassrev10_fix_2_9/PICKUP3_OUT2
- net PICKUP2 renamed /electrobassrev10_fix_2_1/PICKUP2
- net PICKUP2_OUT2 renamed /electrobassrev10_fix_2_9/PICKUP4_OUT2
- net PICKUP2_OUT_HIGH renamed /electrobassrev10_fix_2_8/PICKUP_GND1_HIGH
- net PICKUP3 renamed /electrobassrev10_fix_2_1/PICKUP3
- net PICKUP3_OUT2 renamed /electrobassrev10_fix_2_1/ADC4OPAMPOUT
- net PICKUP3_OUT_HIGH renamed /electrobassrev10_fix_2_9/PICKUP_PWR2
- net PICKUP4 renamed /electrobassrev10_fix_2_1/PICKUP4
- net PICKUP4_OUT renamed /electrobassrev10_fix_2_7/PICKUP_GND1
- net PICKUP_GND1 renamed /electrobassrev10_fix_2_8/PICKUP2_OUT_HIGH
- net PICKUP_GND1_HIGH renamed /electrobassrev10_fix_2_9/PICKUP_GND2
- net PICKUP_GND2 renamed /electrobassrev10_fix_2_9/PICKUP2_OUT2
- net PICKUP_PWR1 renamed /electrobassrev10_fix_2_8/PICKUP_PWR1_HIGH
- net PICKUP_PWR1_HIGH renamed /electrobassrev10_fix_2_8/PICKUP3_OUT_HIGH
- net PICKUP_PWR2 renamed /electrobassrev10_fix_2_9/PICKUP1_OUT2
- net PROG_RESET renamed Net-(IC4-VCCA)
- net PROG_SWDCLK renamed Net-(R52-S)
- net PROG_SWDIO renamed /electrobassrev10_fix_2_1/VCCD_1
- net PROG_SWO renamed Net-(R53-S)
- net SCL renamed /electrobassrev10_fix_2_1/SCL
- net SCLK_1 renamed /electrobassrev10_fix_2_1/SCLK_1
- net SDA renamed /electrobassrev10_fix_2_1/SDA
- net SDA_1 renamed Net-(D13-PadC)
- net SD_CMD renamed /electrobassrev10_fix_2_1/SD_CMD
- net SD_DAT0 renamed /electrobassrev10_fix_2_1/SD_DAT0
- net SD_DAT1 renamed /electrobassrev10_fix_2_1/SD_DAT1
- net SD_DAT2 renamed /electrobassrev10_fix_2_1/SD_DAT2
- net SD_DAT3 renamed /electrobassrev10_fix_2_1/SD_DAT3
- net SPI_READY renamed /electrobassrev10_fix_2_1/SPI_READY
- net SS_1 renamed /electrobassrev10_fix_2_1/SS_1
- net SS_2_P renamed Net-(IC4-P1_2)
- net STRING1_BODY renamed /electrobassrev10_fix_2_1/STRING1_BODY
- net STRING1_NECK renamed /electrobassrev10_fix_2_1/STRING1_NECK
- net STRING2_BODY renamed /electrobassrev10_fix_2_1/STRING2_BODY
- net STRING3_BODY renamed /electrobassrev10_fix_2_1/STRING3_BODY
- net STRING4_BODY renamed /electrobassrev10_fix_2_1/STRING4_BODY
- net STRING4_NECK renamed /electrobassrev10_fix_2_1/STRING4_NECK
- net SWD_CLK_SLIDER renamed /electrobassrev10_fix_2_2/SWD_CLK_SLIDER
- net SWD_IO_SLIDER renamed /electrobassrev10_fix_2_2/SWD_IO_SLIDER
- net SWO_SLIDER renamed /electrobassrev10_fix_2_2/SWO_SLIDER
- net UP renamed /electrobassrev10_fix_2_1/UP
- net USBDM renamed /electrobassrev10_fix_2_1/PROG_SWO
- net USBDP renamed /electrobassrev10_fix_2_1/PROG_SWDCLK
- net VBUS renamed Net-(U5-PDEN)
- net VBUS_DIVIDED renamed /electrobassrev10_fix_2_1/VBUS_DIVIDED
- net VCCA_1 renamed Net-(R47-S)
- net VCCD_1 renamed Net-(R51-S)
- net V_H renamed /electrobassrev10_fix_2_1/V_H
- net V_T renamed /electrobassrev10_fix_2_1/V_T
- net V_T_1 renamed /electrobassrev10_fix_2_1/V_T_1
- net V_T_2 renamed /electrobassrev10_fix_2_1/V_T_2
- net V_T_3 renamed /electrobassrev10_fix_2_1/V_T_3
- net V_T_4 renamed /electrobassrev10_fix_2_1/V_T_4
- net XRES_SLIDER renamed /electrobassrev10_fix_2_2/XRES_SLIDER
- AGND5 pad 1: AGND -> p4b
- C1 pad 2: AGND -> p4b
- C12 pad 2: AGND -> p4b
- C13 pad 2: AGND -> p4b
- C14 pad 2: AGND -> p4b
- C2 pad 2: AGND -> p4b
- C30 pad 2: ADC1OPAMPOUT -> GNDIO
- C31 pad 2: AGND -> p4b
- C32 pad 2: AGND -> p4b
- C33 pad 2: AGND -> p4b
- C34 pad 2: AGND -> p4b
- C41 pad 1: 3V3A1 -> unconnected-(C41-Pad1)
- C41 pad 2: AGND -> p4b
- C42 pad 2: AGND -> p4b
- C47 pad 2: AGND -> p4b
- C5 pad 2: AGND -> p4b
- C51 pad 2: AGND -> p4b
- C52 pad 2: AGND -> p4b
- C53 pad 2: AGND -> p4b
- C55 pad 2: AGND -> p4b
- C57 pad 2: AGND -> p4b
- C58 pad 2: AGND -> p4b
- C59 pad 2: AGND -> p4b
- C6 pad 2: AGND -> p4b
- C60 pad 2: AGND -> p4b
- C62 pad 2: AGND -> p4b
- C64 pad 2: AGND -> p4b
- C65 pad 2: AGND -> p4b
- C7 pad 2: AGND -> p4b
- C8 pad 2: AGND -> p4b
- C87 pad 1: (no net) -> unconnected-(C87-Pad1)
- C9 pad 2: GNDINT -> /electrobassrev10_fix_2_1/ADC2OPAMPOUT
- D1 pad 1: AGND -> p4b
- D2 pad 1: AGND -> p4b
- D20 pad C: N$122 -> 12VD2
- D3 pad 1: AGND -> p4b
- D9 pad 1: AGND -> p4b
- IC1 pad 11: AGND -> p4b
- IC1 pad 7: GNDINT -> /electrobassrev10_fix_2_1/ADC2OPAMPOUT
- IC3 pad 2: AGND -> p4b
- IC4 pad 11: (no net) -> unconnected-(IC4-IND-Pad11)
- IC4 pad 16: (no net) -> Net-(IC4-P5_0)
- IC4 pad 17: (no net) -> Net-(IC4-P5_1)
- IC4 pad 18: (no net) -> Net-(IC4-P5_2)
- IC4 pad 19: (no net) -> Net-(IC4-P5_3)
- IC4 pad 31: (no net) -> unconnected-(IC4-P5_4-Pad31)
- IC4 pad 32: (no net) -> unconnected-(IC4-P5_5-Pad32)
- IC4 pad 33: (no net) -> unconnected-(IC4-P5_6-Pad33)
- IC4 pad 34: (no net) -> unconnected-(IC4-P5_7-Pad34)
- IC4 pad 40: (no net) -> unconnected-(IC4-NC@1-Pad40)
- IC4 pad 41: (no net) -> unconnected-(IC4-NC@2-Pad41)
- IC4 pad 57: (no net) -> unconnected-(IC4-NC@3-Pad57)
- IC4 pad 58: (no net) -> unconnected-(IC4-NC@4-Pad58)
- IC4 pad 59: (no net) -> unconnected-(IC4-NC@5-Pad59)
- IC4 pad 6: (no net) -> unconnected-(IC4-P6_4-Pad6)
- IC4 pad 60: (no net) -> unconnected-(IC4-NC@6-Pad60)
- IC4 pad 61: (no net) -> unconnected-(IC4-NC@7-Pad61)
- IC4 pad 62: (no net) -> unconnected-(IC4-NC@8-Pad62)
- IC4 pad 64: AGND -> p4b
- IC4 pad 7: (no net) -> unconnected-(IC4-P6_5-Pad7)
- IC4 pad 8: (no net) -> unconnected-(IC4-P6_6-Pad8)
- IC4 pad 81: (no net) -> unconnected-(IC4-P4_3-Pad81)
- IC4 pad 82: (no net) -> unconnected-(IC4-P4_4-Pad82)
- IC4 pad 83: (no net) -> unconnected-(IC4-P4_5-Pad83)
- IC4 pad 84: (no net) -> unconnected-(IC4-P4_6-Pad84)
- IC4 pad 85: (no net) -> unconnected-(IC4-P4_7-Pad85)
- IC4 pad 89: (no net) -> unconnected-(IC4-P6_0-Pad89)
- IC4 pad 9: (no net) -> unconnected-(IC4-P6_7-Pad9)
- IC4 pad 90: (no net) -> unconnected-(IC4-P6_1-Pad90)
- IC4 pad 91: (no net) -> unconnected-(IC4-P6_2-Pad91)
- IC4 pad 92: (no net) -> unconnected-(IC4-P6_3-Pad92)
- IC5 pad 2: AGND -> p4b
- J1 pad 1: DAT2 -> Net-(J1-Pin_1)
- J1 pad 2: DAT3 -> GNDINT
- J10 pad 3: AGND -> p4b
- J10 pad 4: AGND -> p4b
- J2 pad 2: AGND -> p4b
- J2 pad 5: AGND -> p4b
- J28 pad 2: N$59 -> DGND3
- J28 pad 3: (no net) -> unconnected-(J28-Pad3)
- J3 pad 2: AGND -> p4b
- J3 pad 5: AGND -> p4b
- J31 pad 1: N$87 -> unconnected-(J31-Pad1)
- J31 pad 2: N$88 -> unconnected-(J31-Pad2)
- J31 pad 3: N$89 -> unconnected-(J31-Pad3)
- J31 pad 4: N$90 -> unconnected-(J31-Pad4)
- J9 pad 3: AGND -> p4b
- J9 pad 4: AGND -> p4b
- JP1 pad 1: N$5 -> unconnected-(JP1-Pad1)
- JP1 pad 2: N$6 -> unconnected-(JP1-Pad2)
- JP1 pad 4: PICKUP4_OUT2 -> GNDINT
- JP1 pad 6: AGND -> p4b
- JP1 pad 7: AGND -> p4b
- JP1 pad 8: ADC1OPAMPOUT -> GNDIO
- JP10 pad 4: (no net) -> unconnected-(JP10-P$4-Pad4)
- JP10 pad 5: SCL_1 -> 3V3D3
- JP10 pad 6: SCL_1 -> 3V3D3
- JP10 pad 7: 3V3D3 -> /electrobassrev10_fix_2_5/O_SDA
- JP11 pad 1: 3V3D3 -> /electrobassrev10_fix_2_5/O_SDA
- JP11 pad 3: SCL_1 -> 3V3D3
- JP15 pad 1: 12VD2 -> Net-(JP15-Pad1)
- JP15 pad 10: N$59 -> DGND3
- JP15 pad 12: N$59 -> DGND3
- JP15 pad 14: N$122 -> 12VD2
- JP15 pad 16: N$122 -> 12VD2
- JP15 pad 3: AGND3 -> Net-(JP15-Pad3)
- JP15 pad 6: N$58 -> AGND3
- JP15 pad 7: N$58 -> AGND3
- JP2 pad 11: STRING2_NECK -> /electrobassrev10_fix_2_1/STRING3_NECK
- JP2 pad 5: STRING3_NECK -> /electrobassrev10_fix_2_1/STRING2_NECK
- JP22 pad 1: (no net) -> unconnected-(JP22-Pad1)
- JP22 pad 4: ADC1OPAMPOUT -> GNDIO
- JP24 pad 10: (no net) -> unconnected-(JP24-P$10-Pad10)
- JP24 pad 3: (no net) -> unconnected-(JP24-P$3-Pad3)
- JP24 pad 4: (no net) -> unconnected-(JP24-P$4-Pad4)
- JP24 pad 8: (no net) -> unconnected-(JP24-P$8-Pad8)
- JP34 pad 1: (no net) -> unconnected-(JP34-P$1-Pad1)
- JP34 pad 3: VDDD_2 -> Net-(JP34-P$3)
- JP34 pad 5: VDDD_2 -> Net-(JP34-P$3)
- JP34 pad 7: VDDD_2 -> Net-(JP34-P$3)
- JP34 pad 8: (no net) -> unconnected-(JP34-P$8-Pad8)
- JP34 pad 9: VDDD_2 -> Net-(JP34-P$3)
- JP5 pad 1: (no net) -> unconnected-(JP5-P$1-Pad1)
- JP5 pad 8: (no net) -> unconnected-(JP5-P$8-Pad8)
- Q1 pad 1: AGND -> p4b
- R118 pad 1: (no net) -> unconnected-(R118-Pad1)
- R118 pad 2: N$2 -> Net-(D15-Pad2)
- R119 pad 1: (no net) -> unconnected-(R119-Pad1)
- R119 pad 2: N$12 -> Net-(D4-Pad2)
- R123 pad 1: (no net) -> unconnected-(R123-Pad1)
- R123 pad 2: N$13 -> Net-(D5-Pad2)
- R124 pad 1: (no net) -> unconnected-(R124-Pad1)
- R124 pad 2: N$14 -> Net-(D6-Pad2)
- R125 pad 1: (no net) -> unconnected-(R125-Pad1)
- R125 pad 2: N$15 -> Net-(D7-Pad2)
- R127 pad 1: DGND3 -> Net-(R127-Pad1)
- R18 pad 1: STRING3_NECK -> /electrobassrev10_fix_2_1/STRING3_NECK
- R19 pad 2: AGND -> p4b
- R192 pad 1: AGND -> p4b
- R199 pad 1: AGND -> p4b
- R20 pad 1: STRING2_NECK -> /electrobassrev10_fix_2_1/STRING2_NECK
- R23 pad 1: RIN3 -> DIST_IN
- R23 pad 2: MONO_STEREO_SWITCH -> Net-(U3-INA-)
- R24 pad 1: GNDINT -> /electrobassrev10_fix_2_1/ADC2OPAMPOUT
- R27 pad 1: A1OUT1 -> DIST_OUT
- R27 pad 2: MONO_STEREO_SWITCH -> Net-(U3-INA-)
- R28 pad 1: A2OUT2 -> Net-(U3-INA-)
- R28 pad 2: MONO_STEREO_SWITCH -> Net-(U3-INB+)
- R29 pad 1: SUM1 -> ADC2_1
- R29 pad 2: MONO_STEREO_SWITCH -> Net-(A6-AUDIO_IN_1)
- R30 pad 1: MONO_STEREO_SWITCH -> ADC3_1
- R30 pad 2: A2OUT1 -> Net-(A2-AUDIO_IN_1)
- R31 pad 1: AGND -> ADC4_1
- R31 pad 2: PICKUP4_OUT2 -> Net-(A3-AUDIO_IN_1)
- R42 pad 1: (no net) -> unconnected-(R42-Pad1)
- R42 pad 2: N$16 -> Net-(D8-Pad2)
- R43 pad 1: (no net) -> unconnected-(R43-Pad1)
- R43 pad 2: N$18 -> Net-(D10-Pad2)
- R44 pad 1: (no net) -> unconnected-(R44-Pad1)
- R44 pad 2: N$32 -> Net-(D11-Pad2)
- R46 pad 2: GNDIO -> Net-(U5-DD+)
- R47 pad 3: AGND -> p4b
- R5 pad 1: SD_CLK -> /electrobassrev10_fix_2_1/SD_CLK
- R50 pad 2: AGND -> p4b
- R51 pad 3: AGND -> p4b
- R52 pad 3: AGND -> p4b
- R53 pad 3: AGND -> p4b
- R58 pad 1: (no net) -> unconnected-(R58-Pad1)
- R58 pad 2: VCCD -> Net-(D12-Pad2)
- R80 pad 2: GNDINT -> /electrobassrev10_fix_2_1/ADC2OPAMPOUT
- U$10 pad P$3: PICKUP4_OUT2 -> GNDINT
- U$10 pad P$6: PICKUP4_OUT2 -> GNDINT
- U1 pad 1: (no net) -> Net-(U1-GPIO0(USB_HS_ID)-Pad1)
- U1 pad 12: (no net) -> Net-(U1-GPIO11(I2C1_SCL)-Pad12)
- U1 pad 13: (no net) -> Net-(U1-GPIO12(I2C1_SDA)-Pad13)
- U1 pad 14: (no net) -> Net-(U1-GPIO13(USART1_TX)-Pad14)
- U1 pad 15: (no net) -> Net-(U1-GPIO14(USART1_RX)-Pad15)
- U1 pad 16: (no net) -> Net-(U1-AUDIO_IN_L-Pad16)
- U1 pad 17: (no net) -> Net-(U1-AUDIO_IN_R-Pad17)
- U1 pad 18: (no net) -> Net-(U1-AUDIO_OUT_L-Pad18)
- U1 pad 19: (no net) -> Net-(U1-AUDIO_OUT_R-Pad19)
- U1 pad 2: (no net) -> Net-(U1-GPIO1(SDMMC1_D3)-Pad2)
- U1 pad 20: AGND -> p4b
- U1 pad 26: (no net) -> Net-(U1-GPIO19(ADC4)-Pad26)
- U1 pad 27: (no net) -> Net-(U1-GPIO20(ADC5)-Pad27)
- U1 pad 28: (no net) -> Net-(U1-GPIO21(ADC6)-Pad28)
- U1 pad 29: (no net) -> Net-(U1-GPIO22(ADC7/DAC2)-Pad29)
- U1 pad 3: (no net) -> Net-(U1-GPIO2(SDMMC1_D2)-Pad3)
- U1 pad 30: (no net) -> Net-(U1-GPIO23(ADC8/DAC1)-Pad30)
- U1 pad 31: (no net) -> Net-(U1-GPIO24(ADC9)-Pad31)
- U1 pad 32: (no net) -> Net-(U1-GPIO25(ADC10)-Pad32)
- U1 pad 33: (no net) -> Net-(U1-GPIO26(SAI2_SD_A)-Pad33)
- U1 pad 34: (no net) -> Net-(U1-GPIO27(SAI2_FS_B)-Pad34)
- U1 pad 35: (no net) -> Net-(U1-GPIO28(ADC11)-Pad35)
- U1 pad 36: (no net) -> Net-(U1-GPIO29(USB_HS_D_-)-Pad36)
- U1 pad 37: (no net) -> Net-(U1-GPIO30(USB_HS_D+)-Pad37)
- U1 pad 4: (no net) -> Net-(U1-GPIO3(SDMMC1_D1)-Pad4)
- U1 pad 5: (no net) -> Net-(U1-GPIO4(SDMMC1_D0)-Pad5)
- U1 pad 6: (no net) -> Net-(U1-GPIO5(SDMMC1_CMD)-Pad6)
- U1 pad B1: (no net) -> Net-(U1-GPIO0(USB_HS_ID)-Pad1)
- U1 pad B12: (no net) -> Net-(U1-GPIO11(I2C1_SCL)-Pad12)
- U1 pad B13: (no net) -> Net-(U1-GPIO12(I2C1_SDA)-Pad13)
- U1 pad B14: (no net) -> Net-(U1-GPIO13(USART1_TX)-Pad14)
- U1 pad B15: (no net) -> Net-(U1-GPIO14(USART1_RX)-Pad15)
- U1 pad B16: (no net) -> Net-(U1-AUDIO_IN_L-Pad16)
- U1 pad B17: (no net) -> Net-(U1-AUDIO_IN_R-Pad17)
- U1 pad B18: (no net) -> Net-(U1-AUDIO_OUT_L-Pad18)
- U1 pad B19: (no net) -> Net-(U1-AUDIO_OUT_R-Pad19)
- U1 pad B2: (no net) -> Net-(U1-GPIO1(SDMMC1_D3)-Pad2)
- U1 pad B20: AGND -> p4b
- U1 pad B26: (no net) -> Net-(U1-GPIO19(ADC4)-Pad26)
- U1 pad B27: (no net) -> Net-(U1-GPIO20(ADC5)-Pad27)
- U1 pad B28: (no net) -> Net-(U1-GPIO21(ADC6)-Pad28)
- U1 pad B29: (no net) -> Net-(U1-GPIO22(ADC7/DAC2)-Pad29)
- U1 pad B3: (no net) -> Net-(U1-GPIO2(SDMMC1_D2)-Pad3)
- U1 pad B30: (no net) -> Net-(U1-GPIO23(ADC8/DAC1)-Pad30)
- U1 pad B31: (no net) -> Net-(U1-GPIO24(ADC9)-Pad31)
- U1 pad B32: (no net) -> Net-(U1-GPIO25(ADC10)-Pad32)
- U1 pad B33: (no net) -> Net-(U1-GPIO26(SAI2_SD_A)-Pad33)
- U1 pad B34: (no net) -> Net-(U1-GPIO27(SAI2_FS_B)-Pad34)
- U1 pad B35: (no net) -> Net-(U1-GPIO28(ADC11)-Pad35)
- U1 pad B36: (no net) -> Net-(U1-GPIO29(USB_HS_D_-)-Pad36)
- U1 pad B37: (no net) -> Net-(U1-GPIO30(USB_HS_D+)-Pad37)
- U1 pad B4: (no net) -> Net-(U1-GPIO3(SDMMC1_D1)-Pad4)
- U1 pad B5: (no net) -> Net-(U1-GPIO4(SDMMC1_D0)-Pad5)
- U1 pad B6: (no net) -> Net-(U1-GPIO5(SDMMC1_CMD)-Pad6)
- U11 pad 14: STRING2_NECK -> /electrobassrev10_fix_2_1/STRING2_NECK
- U11 pad 15: STRING3_NECK -> /electrobassrev10_fix_2_1/STRING3_NECK
- U11 pad 7: AGND -> p4b
- U14 pad 1: (no net) -> unconnected-(U14-P1.7-Pad1)
- U14 pad 10: (no net) -> unconnected-(U14-VSSD_2-Pad10)
- U14 pad 11: (no net) -> unconnected-(U14-NC_2-Pad11)
- U14 pad 12: (no net) -> unconnected-(U14-P3.0-Pad12)
- U14 pad 13: (no net) -> unconnected-(U14-P3.1_2-Pad13)
- U14 pad 14: (no net) -> unconnected-(U14-P3.1-Pad14)
- U14 pad 15: (no net) -> unconnected-(U14-NC_3-Pad15)
- U14 pad 16: (no net) -> unconnected-(U14-P3.3-Pad16)
- U14 pad 17: (no net) -> unconnected-(U14-P3.4-Pad17)
- U14 pad 18: (no net) -> unconnected-(U14-P3.5-Pad18)
- U14 pad 19: (no net) -> unconnected-(U14-P3.6-Pad19)
- U14 pad 2: (no net) -> unconnected-(U14-P2.0-Pad2)
- U14 pad 20: (no net) -> unconnected-(U14-P3.7-Pad20)
- U14 pad 21: AUDIO_L_PREKNOB -> VDDD_2
- U14 pad 22: (no net) -> unconnected-(U14-P4.0-Pad22)
- U14 pad 23: (no net) -> unconnected-(U14-P4.1-Pad23)
- U14 pad 24: (no net) -> unconnected-(U14-P4.2-Pad24)
- U14 pad 25: (no net) -> unconnected-(U14-P4.3-Pad25)
- U14 pad 26: (no net) -> unconnected-(U14-NC_4-Pad26)
- U14 pad 27: (no net) -> unconnected-(U14-NC-Pad27)
- U14 pad 28: (no net) -> unconnected-(U14-P0.0-Pad28)
- U14 pad 29: (no net) -> unconnected-(U14-P0.1-Pad29)
- U14 pad 3: (no net) -> unconnected-(U14-P2.1-Pad3)
- U14 pad 30: (no net) -> unconnected-(U14-P0.2-Pad30)
- U14 pad 31: (no net) -> unconnected-(U14-P0.3-Pad31)
- U14 pad 32: (no net) -> unconnected-(U14-P0.4-Pad32)
- U14 pad 33: (no net) -> unconnected-(U14-P0.5-Pad33)
- U14 pad 34: (no net) -> unconnected-(U14-P0.6-Pad34)
- U14 pad 35: (no net) -> unconnected-(U14-P0.7-Pad35)
- U14 pad 36: (no net) -> unconnected-(U14-XRES-Pad36)
- U14 pad 37: AUDIO_L_POSTKNOB -> VCCD
- U14 pad 38: (no net) -> unconnected-(U14-VSSD-Pad38)
- U14 pad 39: AUDIO_R_POSTKNOB -> VDDD
- U14 pad 4: (no net) -> unconnected-(U14-P2.2-Pad4)
- U14 pad 40: AUDIO_R_PREKNOB -> VDDA
- U14 pad 41: (no net) -> unconnected-(U14-VSSA-Pad41)
- U14 pad 42: (no net) -> unconnected-(U14-P1.0-Pad42)
- U14 pad 43: (no net) -> unconnected-(U14-P1.1-Pad43)
- U14 pad 44: (no net) -> unconnected-(U14-P1.2-Pad44)
- U14 pad 45: (no net) -> unconnected-(U14-P1.3-Pad45)
- U14 pad 46: (no net) -> unconnected-(U14-P1.4-Pad46)
- U14 pad 47: (no net) -> unconnected-(U14-P1.5-Pad47)
- U14 pad 48: (no net) -> unconnected-(U14-P1.6-Pad48)
- U14 pad 5: (no net) -> unconnected-(U14-P2.3-Pad5)
- U14 pad 6: (no net) -> unconnected-(U14-P2.4-Pad6)
- U14 pad 7: (no net) -> unconnected-(U14-P2.5-Pad7)
- U14 pad 8: (no net) -> unconnected-(U14-P2.6-Pad8)
- U14 pad 9: (no net) -> unconnected-(U14-P2.7-Pad9)
- U2 pad 2: AGND -> p4b
- U3 pad 1: A2OUT1 -> Net-(U3-INB+)
- U3 pad 2: MONO_STEREO_SWITCH -> Net-(U3-INA-)
- U3 pad 3: PICKUP4_OUT2 -> GNDINT
- U3 pad 4: VDDA -> -15V
- U3 pad 5: (no net) -> Net-(U3-INB+)
- U3 pad 6: (no net) -> OUTPUT
- U3 pad 7: (no net) -> OUTPUT
- U3 pad 8: (no net) -> +15V
- U5 pad 10: GNDIO -> Net-(U5-DD+)
- U5 pad 2: ADC1OPAMPOUT -> GNDIO
- U5 pad 8: ADC1OPAMPOUT -> GNDIO
- U6 pad 10: (no net) -> unconnected-(U6-NC_2-Pad10)
- U6 pad 11: (no net) -> unconnected-(U6-NC-Pad11)
- U6 pad 4: (no net) -> unconnected-(U6-INT1-Pad4)
- U6 pad 9: (no net) -> unconnected-(U6-INT2-Pad9)
- U8 pad 10: (no net) -> unconnected-(U8-NC_3-Pad10)
- U8 pad 11: (no net) -> unconnected-(U8-NC-Pad11)
- U8 pad 14: (no net) -> unconnected-(U8-GP2-Pad14)
- U8 pad 15: (no net) -> unconnected-(U8-GP3-Pad15)
- U8 pad 17: (no net) -> unconnected-(U8-GP5-Pad17)
- U8 pad 18: (no net) -> unconnected-(U8-GP6-Pad18)
- U8 pad 19: (no net) -> unconnected-(U8-GP7-Pad19)
- U8 pad 3: (no net) -> unconnected-(U8-A2-Pad3)
- U8 pad 4: (no net) -> unconnected-(U8-A1-Pad4)
- U8 pad 5: (no net) -> unconnected-(U8-A0-Pad5)
- U8 pad 6: (no net) -> unconnected-(U8-*RESET-Pad6)
- U8 pad 7: (no net) -> unconnected-(U8-NC_2-Pad7)
- U8 pad 8: (no net) -> unconnected-(U8-INT-Pad8)
- U9 pad 14: STRING2_NECK -> /electrobassrev10_fix_2_1/STRING2_NECK
- U9 pad 15: STRING3_NECK -> /electrobassrev10_fix_2_1/STRING3_NECK
- U9 pad 7: AGND -> p4b
- VR3 pad P$3: AGND -> p4b
- VR4 pad P$3: AGND -> p4b
- X2 pad R: 12VD2 -> Net-(JP15-Pad1)
- X2 pad RN: (no net) -> unconnected-(X2-PadRN)
- X2 pad SN: (no net) -> unconnected-(X2-PadSN)
- X2 pad TN: (no net) -> unconnected-(X2-PadTN)
- X3 pad RN: (no net) -> unconnected-(X3-PadRN)
- X3 pad S: N$58 -> AGND3
- X3 pad SN: AGND3 -> Net-(JP15-Pad3)
- X3 pad TN: (no net) -> unconnected-(X3-PadTN)
- X4 pad S1: DGND3 -> Net-(R127-Pad1)
- X4 pad S2: DGND3 -> Net-(R127-Pad1)
Routing:
- net AGND: track 180.1 -> 0.00 mm, vias 26 -> 0
- net p4b: track 0.00 -> 172.3 mm, vias 0 -> 25
- net STRING3_NECK: track 99.2 -> 0.00 mm
- net /electrobassrev10_fix_2_1/STRING2_NECK: track 0.00 -> 92.3 mm, vias 0 -> 3
- net /electrobassrev10_fix_2_1/STRING3_NECK: track 0.00 -> 85.9 mm, vias 0 -> 1
- net STRING2_NECK: track 79.8 -> 0.00 mm, vias 3 -> 0
- net /electrobassrev10_fix_2_1/V_T_2: track 15.2 -> 68.7 mm, vias 0 -> 4
- net /electrobassrev10_fix_2_1/NECKSENSE1: track 27.5 -> 69.1 mm, vias 1 -> 2
- net /electrobassrev10_fix_2_5/O_SDA: track 0.00 -> 33.7 mm, vias 0 -> 1
- net Net-(JP15-Pad3): track 0.00 -> 32.3 mm
- net AGND3: track 32.3 -> 3.59 mm
- net /electrobassrev10_fix_2_1/STRING4_NECK: track 46.3 -> 74.2 mm, vias 3 -> 5
- net Net-(JP15-Pad1): track 0.00 -> 27.0 mm
- net N$122: track 25.3 -> 0.00 mm
- net 3V3D3: track 33.7 -> 9.91 mm, vias 1 -> 2
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- added copper zone on In2.Cu, net 3V3D3
- added copper zone on In1.Cu, net AGND3
- added copper zone on In2.Cu, net AGND3
- added copper zone on In2.Cu, net DGND3
- added copper zone on In1.Cu, net GNDINT
- added copper zone on F.Cu, net p4b
- added copper zone on In1.Cu, net p4b
- removed copper zone on F.Cu, net AGND
- removed copper zone on In1.Cu, net AGND
- removed copper zone on In1.Cu, net N$122
- removed copper zone on In1.Cu, net N$58
- removed copper zone on In2.Cu, net N$58
- removed copper zone on In2.Cu, net N$59
- removed copper zone on In1.Cu, net PICKUP4_OUT2
- removed copper zone on In2.Cu, net SCL_1
