File: EAGLE_files/rev10/electrobassrev10_fix_2.kicad_pcb (KiCad board)
At the start: 4 copper layers, 346.6 x 245.1 mm, 325 parts, among them IC1 LMV324?M, IC3 LMV321?M5, IC4 CY8C58LPXXX_USB_4JTAG, IC5 LMV321?M5, J1 Conn_01x02_Pin, J10 4P-2.0, J11 4P-2.0, J12 MEM2075-00-140-01-A, J13 4P-2.0, J18 110990030, J2 SM06B-SRSS-TB(LF)(SN), J28 PJ-066A, J3 SM06B-SRSS-TB(LF)(SN), J31 4P-2.0-90D, J4 4P-2.0, J5 SM06B-SRSS-TB(LF)(SN), J6 SM06B-SRSS-TB(LF)(SN), J7 SM06B-SRSS-TB(LF)(SN), J8 SM06B-SRSS-TB(LF)(SN), J9 4P-2.0, Q1 DMP3099L, SW1 B3F-1025, U1 ES_DAISY_SEED_DOUBLE, U11 MC74HC4052ADTR2GTSSOP-16_ONS-L, U14 CY8C4024AZI-S413TQFP_24AZI-S4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, U17 NJM4580, U18 MCP45HV51T-503E/ST, U19 MCP45HV51T-503E/ST, U2 LP2985, U20 MCP45HV51T-503E/ST, U21 MCP45HV51T-503E/ST, U23 INA2134UA, U24 INA2134UA, U28 OPA1642AIDR, U29 DRV135UA/2K5, U3 OPA1642AIDR, U5 ADUM3160BRWZRW_16_ADI-M, U6 LSM6DSLTR, U8 MCP23008T-E/SS, U9 MC74HC4052ADTR2GTSSOP-16_ONS-L, X1 3P-2MM-TH-MALE, X10 3P-2MM-TH-MALE, X11 3P-2MM-TH-MALE, X12 3P-2MM-TH-MALE, X13 3P-2MM-TH-MALE, X14 3P-2MM-TH-MALE, X15 3P-2MM-TH-MALE, X16 332-02, X17 332-02, X18 332-02, X19 332-02, X2 NRJ6HF2, X3 NRJ6HF2, X4 USB+SHIELD, X5 332-02, X6 332-02, X7 332-02, X8 332-02, X9 3P-2MM-TH-MALE

Commit message: working on 5 string version
Parts:
- added U4: Daisy_Seed2_DFM, Snapeda:DAISY_PATCH_SM, F.Cu at (356.1, 8.38)
