File: EAGLE_files/rev10/electrobassrev10_fix_2.kicad_sch (KiCad schematic)
At the start: 0 parts

Commit message: added new electrobass revision kicad files
Other:
- added sheet distortion (distortion.kicad_sch)
- added sheet synthesis (synthesis.kicad_sch)
Changed lines of the file:
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@@
+	)
+	(sheet
+		(at 25.4 95.25)
+		(size 20.32 7.62)
+		(exclude_from_sim no)
+		(in_bom yes)
+		(on_board yes)
+		(dnp no)
+		(fields_autoplaced yes)
+		(stroke
+			(width 0.1524)
+			(type solid)
+		)
+		(fill
+			(color 0 0 0 0.0000)
+		)
+		(property "Sheetname" "distortion"
+			(at 25.4 94.5384 0)
+			(effects
+				(font
+					(size 1.27 1.27)
+				)
+				(justify left bottom)
+			)
+		)
+		(property "Sheetfile" "distortion.kicad_sch"
+			(at 25.4 103.4546 0)
+			(effects
+				(font
+					(size 1.27 1.27)
+				)
+				(justify left top)
+			)
+		)
+		(instances
+			(project "electrobassrev10_fix_2"
+				(path "/1ef21aac-6bb5-463b-b2e7-8b29a3c9e6a7"
+					(page "11")
+				)
+			)
+		)
 	)
 	(sheet
@@
 				)
 			)
+		)
+	)
+	(sheet
+		(at 74.93 92.71)
+		(size 31.75 12.7)
+		(exclude_from_sim no)
+		(in_bom yes)
+		(on_board yes)
+		(dnp no)
+		(fields_autoplaced yes)
+		(stroke
+			(width 0.1524)
+			(type solid)
+		)
+		(fill
+			(color 0 0 0 0.0000)
+		)
+		(property "Sheetname" "synthesis"
+			(at 74.93 91.9984 0)
+			(effects
+				(font
+					(size 1.27 1.27)
+				)
+				(justify left bottom)
+			)
+		)
+		(property "Sheetfile" "synthesis.kicad_sch"
+			(at 74.93 105.9946 0)
+			(effects
+				(font
+					(size 1.27 1.27)
+				)
+				(justify left top)
+			)
+		)
+		(instances
+			(project "electrobassrev10_fix_2"
+				(path "/1ef21aac-6bb5-463b-b2e7-8b29a3c9e6a7"
+					(page "12")
+				)
+			)
