File: EAGLE_files/rev10/electrobassrev10_fix_2_1.kicad_sch (KiCad schematic)
At the start: 180 parts, among them IC1 LMV324?M, IC3 LMV321?M5, IC4 CY8C58LPXXX_USB_4JTAG, IC5 LMV321?M5, J1 105162-0001, J10 4P-2.0, J11 4P-2.0, J13 4P-2.0, J2 SM06B-SRSS-TB(LF)(SN), J3 SM06B-SRSS-TB(LF)(SN), J31 4P-2.0-90D, J4 4P-2.0, J9 4P-2.0, Q1 DMP3099L, U1 ES_DAISY_SEED_DOUBLE, U11 MC74HC4052ADTR2GTSSOP-16_ONS-L, U13 ES_DAISY_SEED_DOUBLE, U2 LP2985, U4 ES_DAISY_SEED_DOUBLE, U5 ADUM3160BRWZRW_16_ADI-M, U6 LSM6DSLTR, U7 ES_DAISY_SEED_DOUBLE, U9 MC74HC4052ADTR2GTSSOP-16_ONS-L

Commit message: added new electrobass revision kicad files
Parts:
- removed J1: 105162-0001, electrobassrev10_fix_2:105162-0001, symbol electrobassrev10_fix_2-eagle-import:105162-0001
- removed R64: 47R, electrobassrev10_fix_2:R0603, symbol electrobassrev10_fix_2-eagle-import:rcl_334_R-US_R0603
- removed U13, U4, U7, U_12: ES_DAISY_SEED_DOUBLE, electrobassrev10_fix_2:ES_DAISY_SEED_DOUBLE, symbol electrobassrev10_fix_2-eagle-import:ES_DAISY_SEED_DOUBLE
- added J12: MEM2075-00-140-01-A, Snapeda:GCT_MEM2075-00-140-01-A, symbol Snapeda:MEM2075-00-140-01-A
- added S1, S3, S5, S6: TL1105SPF160Q, Snapeda:SW_TL1105SPF160Q, symbol Snapeda:TL1105SPF160Q
Connections:
- net +3V3: now also J12.P4 (VDD)
- net CLK: now also J12.P5 (CLK)
- net CMD: now also J12.P3 (CMD)
- net DAT0: now also J12.P7 (DAT0)
- net DAT1: now also J12.P8 (DAT1)
- net DAT2: now also J12.P1 (DAT2)
- net DAT3: now also J12.P2 (CD/DAT3)
- net DGND: now also J12.P6 (VSS), J12.SH1 (SHIELD), J12.SH2 (SHIELD__1), J12.SH3 (SHIELD__2), J12.SH4 (SHIELD__3), S1.1, S1.2, S3.1, S3.2, S5.1, S5.2, S6.1, S6.2
- net PA1_SD_DETECT: now also J12.P9 (CD)
- net STRING2_NECK: now also JP2.5
- net at IC4.16 (P5_0): now also S1.3, S1.4
- net at IC4.17 (P5_1): now also S3.3, S3.4
- net at IC4.18 (P5_2): now also S5.3, S5.4
- net at IC4.19 (P5_3): now also S6.3, S6.4
