File: EAGLE_files/rev10/electrobassrev10_fix_2_4.kicad_sch (KiCad schematic)
At the start: 35 parts, among them IC2 1253S08-U, IC6 1253S08-U, IC7 1253S08-U, IC8 1253S08-U, U10 DG403DVZTSSOP16_4P50X5P10_INR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, U12 DG403DVZTSSOP16_4P50X5P10_INR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, U15 DG403DVZTSSOP16_4P50X5P10_INR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, U16 DG403DVZTSSOP16_4P50X5P10_INR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, U3 OPA1664AIPWRPW14_TEX-L

Commit message: added new electrobass revision kicad files
Parts:
- removed C15, C16, C17, C18, C19, C20, C21, C22, C23, C24, C25, C28: .1uf, electrobassrev10_fix_2:C0603K, symbol electrobassrev10_fix_2-eagle-import:C-USC0603K
- removed C35, C37, C67, C68: 10uf, electrobassrev10_fix_2:C1206K, symbol electrobassrev10_fix_2-eagle-import:C-EUC1206K
- removed IC2, IC6, IC7, IC8: 1253S08-U, electrobassrev10_fix_2:SOIC127P600X173-8N, symbol electrobassrev10_fix_2-eagle-import:1253S08-U
- removed L2: 2.2uH, electrobassrev10_fix_2:BOURNS_SRP2010, symbol electrobassrev10_fix_2-eagle-import:INDUCTORS
- removed PS1: UWE1215S-3WR3, electrobassrev10_fix_2:CONV_UWE1215S-3WR3, symbol electrobassrev10_fix_2-eagle-import:UWE1215S-3WR3
- removed R23, R27, R28, R29, R30, UNK600R0: 10k, electrobassrev10_fix_2:R0603, symbol electrobassrev10_fix_2-eagle-import:adafruit_R-US_R0603
- removed R31: 5R, electrobassrev10_fix_2:R0603, symbol electrobassrev10_fix_2-eagle-import:adafruit_R-US_R0603
- removed U10, U12, U15, U16: DG403DVZTSSOP16_4P50X5P10_INR-L, electrobassrev10_fix_2:TSSOP16_4P50X5P10_INR-L, symbol electrobassrev10_fix_2-eagle-import:DG403DVZTSSOP16_4P50X5P10_INR-L
- removed U3: OPA1664AIPWRPW14_TEX-L, electrobassrev10_fix_2:PW14_TEX-L, symbol electrobassrev10_fix_2-eagle-import:OPA1664AIPWRPW14_TEX-L
- removed UNK12VD1: PINHD-1X1, electrobassrev10_fix_2:1X01, symbol electrobassrev10_fix_2-eagle-import:PINHD-1X1
Other:
- note removed: "Audio"
